Commit message: fix(yhs): provide provisional base_footprint static edge needed by FAST-LIO odom adapter

File: appliance/assets/yhs_mid360/yhs_mid360_tf_nominal.urdf (robot description, URDF)
Before this commit: robot agt_yhs_mid360_tf_nominal, 5 links, 4 joints
Links:
- added link base_footprint
Joints:
- added joint base_footprint_to_base: type fixed, parent base_footprint, child base_link, origin xyz=0 0 0.1041 rpy=0 0 0
